Commit message: Add files via upload
Fixed lidar

File: src/learnbotics/urdf/lidar.xacro (robot description, xacro)
@@ -41,10 +41,10 @@
       <origin rpy="0 0 0" xyz="0 0 0"/>
       <geometry>
-        <mesh filename="package://learnbotics/meshes/vlp16a.stl" scale="0.5 0.5 0.5"/>
+        <mesh filename="package://learnbotics/meshes/vlp16b.stl" scale="0.5 0.5 0.5"/>
       </geometry>
     </visual>
     <collision>
       <geometry>
-          <mesh filename="package://learnbotics/meshes/vlp16a.stl" scale="0.5 0.5 0.5"/>
+          <mesh filename="package://learnbotics/meshes/vlp16b.stl" scale="0.5 0.5 0.5"/>
       </geometry>
       <!-- <origin rpy="0  0  0" xyz="0       0       0.03585"/>

File: src/learnbotics/urdf/model.urdf (robot description, URDF)
Before this commit: robot RobotC2_0_0, 14 links, 15 joints
Joints:
- joint Robot_to_sensor: origin xyz=-0.06 0.041 0.073 rpy=0 0 0 -> xyz=-0.06 0.041 0.091 rpy=0 -0.0261799 3.14159
- joint base_to_capa: origin xyz=0.062575 -0.038531 0.047 rpy=0 0 0 -> xyz=0.062575 -0.038531 0.0465 rpy=0 0 0
