Commit message: Add files via upload
Added camera and lidar, and ros connection

File: src/learnbotics/urdf/camera.xacro (robot description, xacro)
@@ -16,17 +16,22 @@
         </clip>
       </camera>
-      <plugin name="camera_controller" filename="libgazebo_ros_camera.so">
-        <alwaysOn>true</alwaysOn>
-        <updateRate>0.0</updateRate>
-        <cameraName>diff/camera_top</cameraName>
-        <imageTopicName>image_raw</imageTopicName>
-        <cameraInfoTopicName>camera_info</cameraInfoTopicName>
-        <frameName>Camera</frameName>
-        <hackBaseline>0.07</hackBaseline>
-        <distortionK1>0.0</distortionK1>
-        <distortionK2>0.0</distortionK2>
-        <distortionK3>0.0</distortionK3>
-        <distortionT1>0.0</distortionT1>
-        <distortionT2>0.0</distortionT2>
+      <plugin name="gazebo_light_sensor_plugin" filename="liblight_sensor_plugin.so">
+        <cameraName>camera</cameraName>
+         <alwaysOn>true</alwaysOn>
+         <updateRate>10</updateRate>
+         <imageTopicName>rgb/image_raw</imageTopicName>
+         <depthImageTopicName>depth/image_raw</depthImageTopicName>
+         <pointCloudTopicName>depth/points</pointCloudTopicName>
+         <cameraInfoTopicName>rgb/camera_info</cameraInfoTopicName>
+         <depthImageCameraInfoTopicName>depth/camera_info</depthImageCameraInfoTopicName>
+         <frameName>camera_depth_optical_frame</frameName>
+         <baseline>0.1</baseline>
+         <distortion_k1>0.0</distortion_k1>
+         <distortion_k2>0.0</distortion_k2>
+         <distortion_k3>0.0</distortion_k3>
+         <distortion_t1>0.0</distortion_t1>
+         <distortion_t2>0.0</distortion_t2>
+         <pointCloudCutoff>0.4</pointCloudCutoff>
+         <robotNamespace>/</robotNamespace>
       </plugin>
     </sensor>

File: src/learnbotics/urdf/lidar.xacro (robot description, xacro)
@@ -33,10 +33,8 @@
         </noise>
       </ray>
-    </sensor>
+      </sensor>
   </gazebo>
   <link name="base_sensor">
-  </link>
-  <link name="Lidar">
-    <visual>
+  <visual>
       <origin rpy="0 0 0" xyz="0 0 0"/>
       <geometry>
@@ -59,8 +57,24 @@
     </inertial>
   </link>
-  <joint name="Base_to_Lidar" type="fixed">
+  <link name="Lidar">
+        <inertial>
+      <origin rpy="0 0 0" xyz="0 0 0"/>
+      <mass value="0.1"/>
+      <inertia ixx="0.000909131" iyy="0.000909131" izz="0.001107105" ixy="0" ixz="0" iyz="0"/>
+    </inertial>
+  </link>
+  <joint name="Base_to_Lidar" type="revolute">
     <parent link="base_sensor"/>
     <child link="Lidar"/>
     <origin rpy="0 0 0" xyz="0 0 0"/>
+    <axis xyz="0 0 1"/>
+    <limit effort="-1" lower="-10000000000000000" upper="10000000000000000" velocity="10"/>
   </joint>
+  <gazebo>
+  <plugin name="gazebo_lidar_plugin" filename="libvelodyne_plugin.so">
+  <!-- /home/israel/lidar_ws/devel/lib/libvelodyne_plugin.so -->
+      <test>Base_to_Lidar</test>
+      <velocity>10</velocity>
+      </plugin>
+  </gazebo>
 </robot>
